File: pcb/Ergoslide/Ergoslide.kicad_pcb (KiCad board)
At the start: 2 copper layers, 405 x 119.2 mm, 190 parts

Commit message: Fully route the matrix
Parts:
- moved D13 0.65 mm to (357.2, 41.1)
Routing:
- net /LCol2: track 0.00 -> 176.5 mm, vias 0 -> 6
- net /RCol6: track 0.00 -> 171.8 mm, vias 0 -> 6
- net /LCol3: track 0.00 -> 171.8 mm, vias 0 -> 6
- net /RCol5: track 0.00 -> 169.4 mm, vias 0 -> 6
- net /LCol4: track 0.00 -> 167.0 mm, vias 0 -> 6
- net /RCol4: track 0.00 -> 167.0 mm, vias 0 -> 6
- net /RCol3: track 0.00 -> 167.0 mm, vias 0 -> 6
- net /RCol8: track 0.00 -> 166.6 mm, vias 0 -> 6
- net /LCol1: track 0.00 -> 156.1 mm, vias 0 -> 6
- net /RCol9: track 0.00 -> 147.2 mm
- net /RCol7: track 0.00 -> 145.5 mm, vias 0 -> 4
- net /LCol5: track 0.00 -> 135.7 mm, vias 0 -> 5
- net /LCol6: track 0.00 -> 135.7 mm, vias 0 -> 5
- net /RCol2: track 0.00 -> 135.7 mm, vias 0 -> 5
- net /RRow5: track 83.3 -> 211.9 mm
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Other:
- board size 405 x 119.2 mm -> 409.6 x 123.8 mm

Commit message: Muck about with custom footprints and symbols for the Supermini
Started wiring the Supermini in to the left side matrix
Parts:
- added J1: Conn_01x02_Socket, Connector_JST:JST_PH_S2B-PH-K_1x02_P2.00mm_Horizontal, B.Cu at (221.5, 169.4)
- added J2: Conn_01x02_Socket, Connector_JST:JST_PH_S2B-PH-K_1x02_P2.00mm_Horizontal, B.Cu at (7.14, 28.6)
- added LeftController1: ~, supermini-nrf52840-kicad:SuperMini NRF52840, B.Cu at (38.1, 38.8)
- added RightController1: ~, supermini-nrf52840-kicad:SuperMini NRF52840, F.Cu at (247.7, 176.2)
Routing:
- net /LRow6: track 131.0 -> 235.6 mm, vias 0 -> 1
- net /LRow5: track 161.9 -> 249.5 mm, vias 0 -> 1
- net /LRow4: track 152.4 -> 222.9 mm, vias 0 -> 1
- net /LRow3: track 157.5 -> 211.5 mm, vias 0 -> 1
- net /LRow2: track 157.2 -> 192.6 mm
- net /LRow1: track 114.3 -> 145.0 mm, vias 0 -> 2
- net /MCol2: track 115.5 -> 145.1 mm
- net /MCol1: track 115.5 -> 128.5 mm
Other:
- outline, holes or cut-outs redrawn

Commit message: Clean up pcb directory in Git
Parts:
- added H1: MountingHole, MountingHole:MountingHole_2.2mm_M2, F.Cu at (184.5, 133.3)
- added H2: MountingHole, MountingHole:MountingHole_2.2mm_M2, F.Cu at (177.4, 50.0)
- added H3: MountingHole, MountingHole:MountingHole_2.2mm_M2, F.Cu at (64.3, 131.0)
- added H4: MountingHole, MountingHole:MountingHole_2.2mm_M2, F.Cu at (64.3, 47.6)
- added SW1: Switch, Button_Switch_SMD:Panasonic_EVQPUL_EVQPUC, B.Cu at (23.8, 59.6)
- added SW2: Power Switch, ScottoKeebs_Components:Switch_SSAL220100, B.Cu at (28.0, 27.2)
- added TP1: B- testpoint, TestPoint:TestPoint_Pad_2.0x2.0mm, F.Cu at (33.3, 34.5)
- added TP2: B+ testpoint, TestPoint:TestPoint_Pad_2.0x2.0mm, F.Cu at (33.3, 39.3)
- added TP3: GND testpoint, TestPoint:TestPoint_Pad_2.0x2.0mm, F.Cu at (23.8, 50.0)
- added TP4: RST testpoint, TestPoint:TestPoint_Pad_2.0x2.0mm, F.Cu at (32.1, 50.0)
- moved J2 144.4 mm to (150.2, 48.7)
- moved LeftController1 0.44 mm to (38.1, 39.2)
Connections:
- LeftController1 pad 14: unconnected-(LeftController1-GND-Pad14) -> Net-(LeftController1-GND-Pad14)
- LeftController1 pad 15: unconnected-(LeftController1-RST-Pad15) -> Net-(LeftController1-RST)
- LeftController1 pad 28: Net-(J2-Pin_1) -> Net-(LeftController1-B-)
Routing:
- net /LCol7: track 39.5 -> 208.3 mm
- net /LCol6: track 135.7 -> 282.4 mm
- net Net-(J2-Pin_2): track 0.00 -> 133.8 mm, vias 0 -> 1
- net Net-(J2-Pin_1): track 0.00 -> 133.8 mm, vias 0 -> 2
- net /LCol5: track 135.7 -> 259.8 mm
- net /LCol4: track 167.0 -> 269.1 mm
- net /LCol3: track 171.8 -> 251.3 mm
- net /LCol2: track 176.5 -> 234.0 mm
- net /LCol1: track 156.1 -> 190.9 mm
- net Net-(LeftController1-RST): track 0.00 -> 17.7 mm, vias 0 -> 1
- net Net-(LeftController1-GND-Pad14): track 0.00 -> 16.1 mm, vias 0 -> 1
- net Net-(LeftController1-B-): track 0.00 -> 2.93 mm
- net /LRow1: track 145.0 -> 146.2 mm, vias 2 -> 0
- added copper zone on B.Cu, net (none)
- added copper zone on F.Cu, net (none)
Other:
- board text added: "+"
- board text added: "-"
- board text added: "B+"
- board text added: "B-"
- board text added: "Reset"

Commit message: Add TL3330AF260GQ to the PCB, start wiring up the second half
Parts:
- removed SW2: Power Switch, ScottoKeebs_Components:Switch_SSAL220100
- removed TP1: B- testpoint, TestPoint:TestPoint_Pad_2.0x2.0mm
- removed TP2: B+ testpoint, TestPoint:TestPoint_Pad_2.0x2.0mm
- removed TP3: GND testpoint, TestPoint:TestPoint_Pad_2.0x2.0mm
- removed TP4: RST testpoint, TestPoint:TestPoint_Pad_2.0x2.0mm
- added BTN1: Reset button, TL3330AF260QG:SW_TL3330AF260QG, B.Cu at (203.8, 86.0)
- added BTN2: Soft Off button, TL3330AF260QG:SW_TL3330AF260QG, B.Cu at (203.8, 32.5)
- added BTN3: Reset button, TL3330AF260QG:SW_TL3330AF260QG, F.Cu at (240.4, 41.3)
- added BTN4: Soft Off button, TL3330AF260QG:SW_TL3330AF260QG, F.Cu at (240.4, 47.0)
- added GND1: GND testpoint, TestPoint:TestPoint_Pad_2.0x2.0mm, F.Cu at (200.0, 98.0)
- added GND2: GND2 test point, TestPoint:TestPoint_Pad_2.0x2.0mm, F.Cu at (203.5, 39.0)
- added GND3: GND testpoint, TestPoint:TestPoint_Pad_2.0x2.0mm, F.Cu at (233.5, 40.6)
- added H10: MountingHole, MountingHole:MountingHole_2.2mm_M2, F.Cu at (252.5, 138.0)
- added H11: MountingHole, MountingHole:MountingHole_2.2mm_M2, F.Cu at (409.5, 128.5)
- added H12: MountingHole, MountingHole:MountingHole_2.2mm_M2, F.Cu at (409.2, 47.5)
- added H13: MountingHole, MountingHole:MountingHole_2.2mm_M2, F.Cu at (347.8, 128.5)
- added H14: MountingHole, MountingHole:MountingHole_2.2mm_M2, F.Cu at (366.5, 90.5)
- added H15: MountingHole, MountingHole:MountingHole_2.2mm_M2, F.Cu at (333.0, 47.5)
- added H16: MountingHole, MountingHole:MountingHole_2.2mm_M2, F.Cu at (252.5, 91.0)
- added H5: MountingHole, MountingHole:MountingHole_2.2mm_M2, F.Cu at (124.0, 46.5)
- added H6: MountingHole, MountingHole:MountingHole_2.2mm_M2, F.Cu at (115.5, 130.2)
- added H7: MountingHole, MountingHole:MountingHole_2.2mm_M2, F.Cu at (195.2, 139.0)
- added H8: MountingHole, MountingHole:MountingHole_2.2mm_M2, F.Cu at (191.8, 79.8)
- added H9: MountingHole, MountingHole:MountingHole_2.2mm_M2, F.Cu at (252.8, 38.5)
- added RST1: RST testpoint, TestPoint:TestPoint_Pad_2.0x2.0mm, F.Cu at (200.0, 92.5)
- added RST2: RST testpoint, TestPoint:TestPoint_Pad_2.0x2.0mm, F.Cu at (233.5, 44.6)
- added SOFF1: Soft-Off test point, TestPoint:TestPoint_Pad_2.0x2.0mm, F.Cu at (200.0, 29.5)
- added SOFF2: Soft-Off test point, TestPoint:TestPoint_Pad_2.0x2.0mm, F.Cu at (233.5, 48.7)
- RightController1: footprint supermini-nrf52840-kicad:SuperMini NRF52840 -> supermini-nrf52840-kicad:SimpleMini NRF52840; moved to B.Cu
- SW1: value Switch -> Power Switch; footprint Button_Switch_SMD:Panasonic_EVQPUL_EVQPUC -> Button_Switch_SMD:SW_SPDT_CK_JS102011SAQN
- moved SW1 180.0 mm to (203.2, 46.0)
- moved H1 163.3 mm to (43.0, 52.0)
- moved LeftController1 150.4 mm to (187.1, 59.7), turned to 90 degrees
- moved J2 117.4 mm to (251.3, 108.2)
- moved RightController1 116.9 mm to (264.5, 60.5), turned to -90 degrees
- moved J1 86.3 mm to (192.9, 88.0), turned to 90 degrees
- moved H4 52.1 mm to (94.2, 90.2)
- moved H3 21.7 mm to (42.8, 128.5)
- moved H2 16.2 mm to (193.5, 48.2)
- moved D10 3.20 mm to (299.0, 38.1)
- moved D13 3.20 mm to (356.1, 38.1)
- moved D14 3.20 mm to (375.2, 38.1)
- moved D15 3.20 mm to (394.2, 38.1)
- moved D39 3.20 mm to (137.1, 81.0)
- moved D45 3.20 mm to (308.5, 81.0)
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Connections:
- J1 pad 1: unconnected-(J1-Pin_1-Pad1) -> Net-(J1-Pin_1)
- J1 pad 2: unconnected-(J1-Pin_2-Pad2) -> Net-(J1-Pin_2)
- LeftController1 pad 12: unconnected-(LeftController1-D9_P1.06-Pad12) -> Net-(LeftController1-D9_P1.06)
- LeftController1 pad 14: Net-(LeftController1-GND-Pad14) -> Net-(BTN1-Pad1)
- LeftController1 pad 17: /MCol1 -> /LRow6
- LeftController1 pad 18: /MCol2 -> /LRow5
- LeftController1 pad 19: /LRow1 -> /LRow4
- LeftController1 pad 20: /LRow2 -> /LRow3
- LeftController1 pad 21: /LRow3 -> /LRow2
- LeftController1 pad 22: /LRow4 -> /LRow1
- LeftController1 pad 23: /LRow5 -> /MCol1
- LeftController1 pad 24: /LRow6 -> /MCol2
- LeftController1 pad 29: Net-(J2-Pin_2) -> Net-(J1-Pin_2)
- LeftController1 pad 3: unconnected-(LeftController1-GND-Pad3) -> Net-(BTN2-Pad2)
- RightController1 pad 10: unconnected-(RightController1-D6_P1.00-Pad10) -> /RCol6
- RightController1 pad 11: unconnected-(RightController1-D7_P0.11-Pad11) -> /RCol7
- RightController1 pad 12: unconnected-(RightController1-D8_P1.04-Pad12) -> /RCol8
- RightController1 pad 14: unconnected-(RightController1-D10_P0.09-Pad14) -> Net-(BTN3-Pad1)
- RightController1 pad 15: unconnected-(RightController1-D16_P0.10-Pad15) -> Net-(RightController1-RST)
- RightController1 pad 17: unconnected-(RightController1-D15_P1.13-Pad17) -> Net-(RightController1-D21_P0.31)
- RightController1 pad 18: unconnected-(RightController1-D18_P1.15-Pad18) -> /RRow1
- RightController1 pad 19: unconnected-(RightController1-D19_P0.02-Pad19) -> /RRow2
- RightController1 pad 20: unconnected-(RightController1-D20_P0.29-Pad20) -> /RRow3
- RightController1 pad 21: unconnected-(RightController1-D21_P0.31-Pad21) -> /RRow4
- RightController1 pad 22: unconnected-(RightController1-3.3V-Pad22) -> /RRow5
- RightController1 pad 23: unconnected-(RightController1-RST-Pad23) -> /RRow6
- RightController1 pad 24: unconnected-(RightController1-GND-Pad24) -> /RCol9
- RightController1 pad 28: unconnected-(RightController1-P1.02-Pad28) -> Net-(J2-Pin_1)
- RightController1 pad 29: unconnected-(RightController1-P1.07-Pad29) -> Net-(J2-Pin_2)
- RightController1 pad 5: unconnected-(RightController1-GND-Pad5) -> /RCol1
- RightController1 pad 6: unconnected-(RightController1-D2_P0.17-Pad6) -> /RCol2
- RightController1 pad 7: unconnected-(RightController1-D3_P0.20-Pad7) -> /RCol3
- RightController1 pad 8: unconnected-(RightController1-D4_P0.22-Pad8) -> /RCol4
- RightController1 pad 9: unconnected-(RightController1-D5_P0.24-Pad9) -> /RCol5
- SW1 pad 1: Net-(LeftController1-GND-Pad14) -> Net-(J1-Pin_1)
- SW1 pad 2: Net-(LeftController1-RST) -> Net-(LeftController1-B-)
Routing:
- net /LCol3: track 251.3 -> 751.0 mm, vias 6 -> 1
- net /LCol4: track 269.1 -> 722.0 mm, vias 6 -> 1
- net /LCol2: track 234.0 -> 637.8 mm, vias 6 -> 1
- net /MCol1: track 128.5 -> 499.9 mm, vias 5 -> 1
- net /LCol1: track 190.9 -> 542.5 mm, vias 6 -> 1
- net /MCol2: track 145.1 -> 475.5 mm, vias 5 -> 1
- net /LCol5: track 259.8 -> 574.3 mm, vias 5 -> 1
- net /LCol7: track 208.3 -> 32.5 mm, vias 2 -> 0
- net /RRow2: track 152.4 -> 0.00 mm
- net Net-(J2-Pin_2): track 133.8 -> 0.00 mm, vias 1 -> 0
- net Net-(J2-Pin_1): track 133.8 -> 0.00 mm, vias 2 -> 0
- net /RCol9: track 147.2 -> 262.8 mm, vias 0 -> 1
- net /RRow1: track 152.4 -> 267.9 mm
- net /RCol1: track 102.1 -> 0.00 mm, vias 4 -> 0
- net /RCol8: track 166.6 -> 235.0 mm, vias 6 -> 2
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- removed copper zone on B.Cu, net (none)
- removed copper zone on F.Cu, net (none)
Other:
- board outline removed
- board text removed: "+"
- board text removed: "-"
- board text removed: "B+"
- board text removed: "B-"
- board text removed: "Reset"

Commit message: Finish wiring up right hand side PCB
Parts:
- added SW2: SW_SPDT, Button_Switch_SMD:SW_SPDT_CK_JS102011SAQN, B.Cu at (245.0, 42.5)
- BTN3, BTN4: moved to B.Cu
- moved RST2 69.6 mm to (247.8, 112.8)
- moved BTN3 53.4 mm to (244.9, 94.5), turned to 90 degrees
- moved SOFF2 23.7 mm to (250.8, 32.5)
- moved H4 23.3 mm to (71.2, 87.1)
- moved GND3 22.0 mm to (250.8, 27.0)
- moved BTN4 18.6 mm to (244.9, 29.0), turned to 90 degrees
- moved H14 12.2 mm to (377.9, 86.2)
- moved GND1 9.78 mm to (200.8, 88.2)
- moved BTN1 8.61 mm to (205.1, 94.5)
- moved RightController1 5.49 mm to (260.1, 57.1)
- moved D89 5.10 mm to (273.7, 134.8)
- moved D90 5.10 mm to (307.1, 134.8)
- moved D92 5.10 mm to (349.9, 134.8)
- moved D94 5.10 mm to (390.4, 134.8)
- moved D95 5.10 mm to (409.4, 134.8)
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Connections:
- RightController1 pad 29: Net-(J2-Pin_2) -> Net-(RightController1-B+)
Routing:
- net /RRow2: track 0.00 -> 180.1 mm, vias 0 -> 9
- net /RRow6: track 152.7 -> 274.2 mm, vias 0 -> 1
- net /RRow5: track 163.0 -> 283.1 mm, vias 8 -> 9
- net /RRow3: track 184.9 -> 273.2 mm, vias 9 -> 10
- net /RRow4: track 177.1 -> 264.3 mm, vias 8 -> 9
- net Net-(BTN3-Pad1): track 0.00 -> 78.8 mm, vias 0 -> 3
- net /RCol1: track 0.00 -> 73.8 mm
- net Net-(J2-Pin_2): track 0.00 -> 73.5 mm
- net Net-(RightController1-RST): track 0.00 -> 69.5 mm, vias 0 -> 2
- net Net-(J2-Pin_1): track 0.00 -> 41.8 mm
- net Net-(RightController1-D21_P0.31): track 0.00 -> 27.6 mm, vias 0 -> 1
- net /LCol2: track 637.8 -> 662.5 mm
- net Net-(RightController1-B+): track 0.00 -> 7.95 mm
- net Net-(LeftController1-RST): track 30.9 -> 38.7 mm
- net Net-(BTN1-Pad1): track 36.2 -> 34.9 mm
