File: pcb/Ergoslide/Ergoslide.kicad_pcb (KiCad board)
At the start: 2 copper layers, 223 parts, among them J1 Conn_01x02_Socket, J2 Conn_01x02_Socket, SW1 Power Switch, SW2 SW_SPDT

Commit message: Add fill zones
Routing:
- added copper zone on B.Cu, net (none)
- added copper zone on F.Cu, net (none)
Other:
- board outline added: 400 x 120 mm
Changed lines of the file:
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@@
 		(tags "test point SMD pad rectangle square")
 		(property "Reference" "GND3"
-			(at 0 -1.998 0)
+			(at -3.75 -1.5 0)
 			(layer "F.SilkS")
 			(effects
@@
 		)
 		(fp_text user "${REFERENCE}"
-			(at 0 -2 0)
+			(at -3.75 -1.5 0)
 			(layer "F.Fab")
 			(effects
@@
 		(net 135)
 	)
+	(gr_rect
+		(start 25 24.5)
+		(end 207 144.5)
+		(stroke
+			(width 0.05)
+			(type solid)
+		)
+		(fill no)
+		(layer "Edge.Cuts")
+	)
+	(gr_rect
+		(start 243 24.5)
+		(end 425 144.5)
+		(stroke
+			(width 0.05)
+			(type solid)
+		)
+		(fill no)
+		(layer "Edge.Cuts")
+	)
 	(segment
 		(start 179.609375 64.453125)
@@
 		(net 149)
 	)
+	(zone
+		(net 0)
+		(net_name "")
+		(layers "F.Cu" "B.Cu")
+		(hatch edge 0.5)
+		(priority 1)
+		(connect_pads
+			(clearance 0.5)
+		)
+		(min_thickness 0.25)
+		(filled_areas_thickness no)
+		(fill yes
+			(thermal_gap 0.5)
+			(thermal_bridge_width 0.5)
+			(island_removal_mode 1)
+			(island_area_min 10)
+		)
+		(polygon
+			(pts
+				(xy 241.25 22.5) (xy 429.5 21.25) (xy 428 146.75) (xy 238.5 149.25) (xy 235.75 25.25)
+			)
+		)
+	)
+	(zone
+		(net 0)
+		(net_name "")
+		(layers "F.Cu" "B.Cu")
+		(hatch edge 0.5)
+		(connect_pads
+			(clearance 0.5)
+		)
+		(min_thickness 0.25)
+		(filled_areas_thickness no)
+		(fill yes
+			(thermal_gap 0.5)
+			(thermal_bridge_width 0.5)
+			(island_removal_mode 1)
+			(island_area_min 10)
+		)
+		(polygon
+			(pts
+				(xy 64.25 21.75) (xy 74.25 22.75) (xy 211.75 22.75) (xy 209.75 150.25) (xy 21.5 150.25) (xy 22.5 20.5)
+				(xy 53.5 20.5) (xy 57 21.25)
+			)
+		)
+	)
 	(embedded_fonts no)

Commit message: Use stabilized switch cutouts
Parts:
- S65, S69, S89: footprint Gateron_KS33_Hotswap:Gateron-KS33-Hotswap-2.25U -> Gateron_KS33_Hotswap:Gateron-KS33-Hotswap-2.25U Stabilized
- S88: footprint Gateron_KS33_Hotswap:Gateron-KS33-Hotswap-2.75U -> Gateron_KS33_Hotswap:Gateron-KS33-Hotswap-2.75U Stabilized
Routing:
- net /LRow5: track 250.8 -> 356.8 mm
- net /RRow4: track 264.3 -> 292.6 mm
- net /LRow6: track 259.1 -> 281.2 mm
- net /RRow5: track 283.1 -> 269.7 mm
- net /RCol8: track 235.0 -> 240.7 mm
- net /RCol7: track 210.5 -> 216.2 mm
- net /RRow6: track 274.2 -> 274.0 mm, vias 1 -> 3
Other:
- board size 400 x 120 mm -> 400 x 122 mm

Commit message: Add Caps Lock LED, remove labels for holes, realign labels for everything else
Parts:
- added D96: LED, LED_SMD:LED_0603_1608Metric, F.Cu at (65.8, 96.8)
- added R1: Resistor, Resistor_SMD:R_0603_1608Metric, F.Cu at (65.8, 93.2)
Connections:
- LeftController1 pad 1: unconnected-(LeftController1-D1_P0.06-Pad1) -> Net-(LeftController1-D1_P0.06)
Routing:
- net Net-(LeftController1-D1_P0.06): track 0.00 -> 183.6 mm, vias 0 -> 5
- net Net-(D96-K): track 34.9 -> 175.1 mm, vias 1 -> 3
- net Net-(D96-A): track 0.00 -> 3.67 mm
