File: pcb/Ergoslide/Ergoslide.kicad_pcb (KiCad board)
At the start: 2 copper layers, 400 x 122 mm, 225 parts, among them J1 Conn_01x02_Socket, J2 Conn_01x02_Socket, SW1 Power Switch, SW2 SW_SPDT

Commit message: Add some tacky text saying who made this thing
Other:
- board text added: "Designed by Michael Hudson"
- board text added: "Ergoslide v1.0"
